File: power_supply.sch (KiCad schematic (older format))
At the start: 39 parts, among them P1 CONN_01X02, P2 CONN_01X03, T1 TRANSFO_2-2, U1 LM317AT, U2 LM337T

Commit message: Updated components ref
Parts:
- removed C9: 47n, Capacitors_ThroughHole:C_Rect_L7_W4.5_P5, symbol C
- removed D10: LED, LEDs:LED-3MM, symbol LED
- added C101: 47n, Capacitors_ThroughHole:C_Rect_L7_W4.5_P5, symbol C
- added D10: LED, LEDs:LED-5MM, symbol LED-RESCUE-power_supply
- added P101: CONN_01X02, CONN:CONN_2, symbol CONN_01X02
- C1, C4: Description (none) -> Condensateurs électrolytiques aluminium – traversant 63volt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; Distributor (none) -> Mouser; Distributor Part # (none) -> 647-UVR1J222MHD; Manufacturer (none) -> Nichicon; Mfg_Part_# (none) -> UVR1J222MHD; Package (none) -> 2-THT
- C10, C7, C8: Description (none) -> Condensateurs à film 100volts 0.047uF; Distributor (none) -> Mouser; Distributor Part # (none) -> 647-QYX2A473KTP; Manufacturer (none) -> Nichicon; Mfg_Part_# (none) -> QYX2A473KTP; Package (none) -> 2-THT
- C11, C12, C13, C14: Description (none) -> Condensateurs à film 100volts 0.1uF; Distributor (none) -> Mouser; Distributor Part # (none) -> 647-QYX2A104KTP; Manufacturer (none) -> Nichicon; Mfg_Part_# (none) -> QYX2A104KTP; Package (none) -> 2-THT
- C2, C5: footprint Capacitors_ThroughHole:C_Radial_D5_L11_P2 -> Capacitors_THT:CP_Radial_D10.0mm_P3.50mm; Description (none) -> Condensateurs électrolytiques aluminium – traversant 50volt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; Distributor (none) -> Mouser; Distributor Part # (none) -> 647-UVR1H101MPD; Manufacturer (none) -> Nichicon; Mfg_Part_# (none) -> UVR1H101MPD; Mfg_Part_No TVX1E101MAD -> UVR1H101MPD; Package (none) -> 2-THT
- C3, C6: Description (none) -> Condensateurs électrolytiques aluminium – traversant 50volt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; Distributor (none) -> Mouser; Distributor Part # (none) -> 647-UPW1H220MDD; Manufacturer (none) -> Nichicon; Mfg_Part_# (none) -> UPW1H220MDD; Mfg_Part_No UVR1E220MDD -> UPW1H220MDD; Package (none) -> 2-THT
- D1, D2, D3, D4: Description (none) -> Redresseurs 3.0 Amp 1300 Volt; Distributor (none) -> Mouser; Distributor Part # (none) -> 625-BY255P-E3; Manufacturer (none) -> Vishay Semiconductors; Mfg_Part_# (none) -> BY255P-E3/54; Mfg_Part_No BY255P-E3/54 BY255P-E3/54 -> BY255P-E3/54; Package (none) -> DO-201AD
- D5, D6, D7, D8: footprint Diodes_ThroughHole:Diode_DO-35_SOD27_Horizontal_RM10 -> Diodes_THT:Diode_DO-41_SOD81_Horizontal_RM10; Description (none) -> Redresseurs Vr/1000V Io/1A T/R; Distributor (none) -> Mouser; Distributor Part # (none) -> 621-1N4007; Manufacturer (none) -> Diodes Incorporated; Mfg_Part_# (none) -> 1N4007-T; Mfg_Part_No 1N4007 -> 1N4007-T; Package (none) -> DO-41
- D9: footprint LEDs:LED-3MM -> LEDs:LED-5MM; symbol LED -> LED-RESCUE-power_supply; Description (none) -> DEL standard - Trou traversant Pink Clear 2200mcd; Distributor (none) -> Mouser; Distributor Part # (none) -> 696-SSL-LX5093PC; Manufacturer (none) -> Lumex; Mfg_Part_# (none) -> SSL-LX5093PC; Package (none) -> T-1 3/4 5mm
- F1: Description (none) -> Accessoires pour supports de fusibles FAC/FAU FUSE CARRIER; Distributor (none) -> Mouser; Distributor Part # (none) -> 693-0031.1666; Manufacturer (none) -> Schurter; Mfg_Part_# (none) -> 0031.1666; Package (none) -> Panel
- P1: Description (none) -> Borniers fixes WR-TBL Model 101 2Pin 5mm Hztl; Distributor (none) -> Mouser; Distributor Part # (none) -> 710-691101710002; Manufacturer (none) -> Wurth Electronics; Mfg_Part_# (none) -> 691101710002; Mfg_Part_No PX0580/28 -> 691101710002; Package (none) -> 2-THT
- P2: Description (none) -> Borniers fixes WR-TBL Md101 5mm VDE 3Pin Hrztl EntryMdlr; Distributor (none) -> Mouser; Distributor Part # (none) -> 710-691101710003; Manufacturer (none) -> Wurth Electronics; Mfg_Part_# (none) -> 691101710003; Package (none) -> 3-THT
- R1, R4: footprint Resistors_ThroughHole:Resistor_Horizontal_RM7mm -> Resistors_THT:R_Axial_DIN0204_L3.6mm_D1.6mm_P5.08mm_Horizontal; Description (none) -> Résistances à couche métallique - Trou traversant 1/3watts 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; Distributor (none) -> Mouser; Distributor Part # (none) -> 71-CCF50-221; Manufacturer (none) -> Vishay / Dale; Mfg_Part_# (none) -> CCF50221RFKR36; Mfg_Part_No 0 -> CCF50221RFKR36; Package (none) -> 2-THT
- R2, R5: footprint Resistors_ThroughHole:Resistor_Horizontal_RM7mm -> Resistors_THT:R_Axial_DIN0207_L6.3mm_D2.5mm_P10.16mm_Horizontal; Description (none) -> Résistances à couche métallique - Trou traversant 400mW 2.2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; Distributor (none) -> Mouser; Distributor Part # (none) -> 594-5043ED2K200F; Manufacturer (none) -> Vishay / BC Components; Mfg_Part_# (none) -> SFR2500002201FR500; Mfg_Part_No CCF072K20JKE36 -> SFR2500002201FR500; Package (none) -> 2-THT
- R21, R51: footprint Resistors_ThroughHole:Resistor_Horizontal_RM7mm -> Resistors_THT:R_Axial_DIN0309_L9.0mm_D3.2mm_P12.70mm_Horizontal; Description (none) -> Résistances à couche métallique - Trou traversant 1/8watt 2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; Distributor (none) -> Mouser; Distributor Part # (none) -> 71-RN60C2200B; Manufacturer (none) -> Vishay / Dale; Mfg_Part_# (none) -> RN60C2200BB14; Package (none) -> DIN0309
- R3: value 1K -> 4.7K; footprint Resistors_ThroughHole:Resistor_Horizontal_RM7mm -> Resistors_THT:R_Axial_DIN0207_L6.3mm_D2.5mm_P10.16mm_Horizontal; Description (none) -> Résistances à couche métallique - Trou traversant 1/4watt 4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; Distributor (none) -> Mouser; Distributor Part # (none) -> 71-CCF07-J-4.7K-E3; Manufacturer (none) -> Vishay / Dale; Mfg_Part_# (none) -> CCF074K70JKE36; Package (none) -> DIN0207
- R6: value 1K -> 4.7K; footprint Resistors_ThroughHole:Resistor_Horizontal_RM7mm -> Resistors_THT:R_Axial_DIN0207_L6.3mm_D2.5mm_P10.16mm_Horizontal; Description (none) -> Résistances à couche métallique - Trou traversant 1/4watt 4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; Distributor (none) -> Mouser; Distributor Part # (none) -> 71-CCF07-J-4.7K-E3; Manufacturer (none) -> Vishay / Dale; Mfg_Part_# (none) -> CCF074K70JKE36; Mfg_Part_No 0 -> (none); Package (none) -> DIN0207
- T1: Description (none) -> Transformateurs d'alimentation PC, Class 2/3, 20VA 36V CT@0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; Distributor (none) -> Mouser; Distributor Part # (none) -> 553-FS36-550-C2; Manufacturer (none) -> Triad Magnetics; Mfg_Part_# (none) -> FS36-550-C2; Mfg_Part_No FS36-550-C2 FS36-550-C2 FS36-550-C2 -> FS36-550-C2; Package (none) -> 8-THT
- U1: Description (none) -> Régulateurs de tension linéaires 3/4 Pin 1.5A Adj Pos Vltg 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; Distributor (none) -> Mouser; Distributor Part # (none) -> 595-LM317KCSE3; Manufacturer (none) -> Texas Instruments; Mfg_Part_# (none) -> LM317KCSE3; Mfg_Part_No LM317KCSE3 LM317KCSE3 -> LM317KCSE3; Package (none) -> TO-220-3
- U2: Description (none) -> Régulateurs de tension linéaires 3-TERMINAL ADJ NEG REG; Distributor (none) -> Mouser; Distributor Part # (none) -> 926-LM337T/NOPB; Manufacturer (none) -> Texas Instruments; Mfg_Part_# (none) -> LM337T/NOPB; Package (none) -> TO-220-3
- VR1: Description (none) -> Varistances 250V 1000pF; Distributor (none) -> Mouser; Distributor Part # (none) -> 576-V250LA40AP; Manufacturer (none) -> Littelfuse; Mfg_Part_# (none) -> V250LA40AP; Package (none) -> 2-THT
Connections:
- net -15V: now also D10.1 (K)
- net AC_1: now also P101.1 (P1); no longer F1.1
- net at T1.1 (PA), VR1.1: now also P101.2 (P2); no longer F1.2
- net at C10.1, C8.2, D2.2 (A)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: now also C101.1
- net at C10.2, C12.2, C4.2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: now also C101.2
- net at R6.2: now also D10.2 (A)
- no-connect marks 0 -> 2
Other:
- moved on the sheet: F1
